File: motor controller.kicad_pcb (KiCad board)
At the start: 2 copper layers, 38 x 18 mm, 27 parts, among them IC1 MA702, IC2 MC33926PNB, IC3 LP38690SD-ADJ_NOPB, J1 Conn_01x06_Male, J2 Conn_01x06_Male, J3 Conn_01x04_Male, M1 Motor_DC, U1 STM32L432KCUx, Y1 32mhz

Commit message: V2
Parts:
- turned IC1 to 180 degrees
Connections:
- IC1 pad 9: Net-(IC1-Pad9) -> (no net)
- R5 pad 2: GND -> IN2
- R6 pad 2: +3V3 -> IN1
- U1 pad 15: D2 -> IN2
- U1 pad 22: Net-(U1-Pad22) -> D2
- U1 pad 25: D1 -> IN1
- U1 pad 26: Net-(U1-Pad26) -> D1
Routing:
- net IN2: track 0.00 -> 27.2 mm, vias 0 -> 4
- net IN1: track 0.00 -> 20.9 mm, vias 0 -> 5
- net +3V3: track 52.8 -> 37.9 mm, vias 11 -> 9
- net SCK: track 19.4 -> 25.7 mm, vias 4 -> 3
- net MISO: track 24.8 -> 29.0 mm, vias 2 -> 5
- net GND: track 55.6 -> 52.1 mm, vias 134 -> 131
- net ENC_CS: track 6.80 -> 7.78 mm
- net MOSI: track 23.1 -> 22.1 mm
- net D2: track 15.0 -> 14.3 mm, vias 3 -> 1
