File: motor controller.sch (KiCad schematic (older format))
At the start: 27 parts, among them IC1 MA702, IC2 MC33926PNB, IC3 LP38690SD-ADJ_NOPB, J1 Conn_01x06_Male, J2 Conn_01x06_Male, J3 Conn_01x04_Male, M1 Motor_DC, U1 STM32L432KCUx, Y1 32mhz

Commit message: V2
Connections:
- net labels added: IN1, IN2
Changed lines of the file:
@@
 EESchema Schematic File Version 4
+LIBS:motor controller-cache
 EELAYER 26 0
 EELAYER END
@@
 Text GLabel 6350 4350 3    50   Input ~ 0
 D2
-$Comp
-L power:+3.3V #PWR0120
-U 1 1 5B3B2BEA
-P 5050 2750
-F 0 "#PWR0120" H 5050 2600 50  0001 C CNN
-F 1 "+3.3V" V 5065 2878 50  0000 L CNN
-F 2 "" H 5050 2750 50  0001 C CNN
-F 3 "" H 5050 2750 50  0001 C CNN
-	1    5050 2750
-	0    -1   -1   0
-$EndComp
-$Comp
-L power:GND #PWR0121
-U 1 1 5B3B2C4A
-P 5050 2650
-F 0 "#PWR0121" H 5050 2400 50  0001 C CNN
-F 1 "GND" V 5055 2522 50  0000 R CNN
-F 2 "" H 5050 2650 50  0001 C CNN
-F 3 "" H 5050 2650 50  0001 C CNN
-	1    5050 2650
-	0    1    1    0
-$EndComp
 Text GLabel 5950 1750 1    50   Input ~ 0
 OUT2
@@
 Text GLabel 3050 3650 2    50   Input ~ 0
 SWCLK
-Text GLabel 2050 3250 0    50   Input ~ 0
+Text GLabel 3050 3450 2    50   Input ~ 0
 D2
-Text GLabel 3050 3750 2    50   Input ~ 0
+Text GLabel 2050 3350 0    50   Input ~ 0
 D1
 $Comp
@@
 	1    0    0    -1
 $EndComp
+Text GLabel 5050 2650 0    50   Input ~ 0
+IN2
+Text GLabel 5050 2750 0    50   Input ~ 0
+IN1
+Text GLabel 3050 3750 2    50   Input ~ 0
+IN1
+Text GLabel 2050 3250 0    50   Input ~ 0
+IN2
 $EndSCHEMATC
