File: motor controller Mini(SPI)/motor controller.sch (KiCad schematic (older format))
At the start: 29 parts, among them IC1 MA702, IC2 ACS711KEXLT-15AB-T, IC3 MIC5501-3.0YM5-TR, IC4 A3918SESTR-T, J1 Conn_01x06_Male, J2 Conn_01x06_Male, J3 Conn_01x04_Male, M1 Motor_DC, U1 STM32L432KCUx, Y1 32mhz

Commit message: Push to new server
Parts:
- removed C12: 10Uf, Capacitor_SMD:C_0805_2012Metric, symbol Device:C
- removed C4, C5: 0.1Uf, Capacitor_SMD:C_0201_0603Metric, symbol Device:C
- removed D1: LED, LED_SMD:LED_0201_0603Metric, symbol Device:LED
- removed IC2: ACS711KEXLT-15AB-T, ACS711KEXLT-15AB-T:EX-PACKAGE, symbol ACS711KEXLT-15AB-T:ACS711KEXLT-15AB-T
- removed IC4: A3918SESTR-T, A3918SESTR-T:QFN50P300X300X80-17N-D, symbol A3918SESTR-T:A3918SESTR-T
- removed J1: Conn_01x06_Male, Connector_PinHeader_1.00mm:PinHeader_1x06_P1.00mm_Vertical, symbol Connector:Conn_01x06_Male
- removed R5, R6: 10K, Resistor_SMD:R_0201_0603Metric, symbol Device:R
- removed Y1: 32mhz, ECX-31B:ECX-1247, symbol Device:Crystal_GND24
- added FB1, FB2: Ferrite_Bead, Inductor_SMD:L_0603_1608Metric, symbol Device:Ferrite_Bead
- added IC4: DRV8837CDSGT, DRV8837CDSGT:SON50P200X200X80-9N, symbol DRV8837CDSGT:DRV8837CDSGT
- C1, C2: value 10pF -> 0.1uF
- C10, C11: value 0.1Uf -> 100nF
- C3, C8, C9: value 1UF -> 1uF
- C6: value 0.1Uf -> 0.1UuF
- C7: value 0.1Uf -> 47pF; footprint Capacitor_SMD:C_0201_0603Metric -> Capacitor_SMD:C_0402_1005Metric
- J2: footprint Connector_PinHeader_1.00mm:PinHeader_1x06_P1.00mm_Vertical -> Connector_Molex:Molex_CLIK-Mate_502386-0670_1x06-1MP_P1.25mm_Horizontal
- M1: footprint hv5932mgMotor:hv5932mgMotor -> mg92b:mg92b
- R2: value 600 -> 1k
- R3: value 10K -> 550
- R4: value 10K -> 0.33; footprint Resistor_SMD:R_0201_0603Metric -> Resistor_SMD:R_0805_2012Metric
Connections:
- net labels added: PREF, SCK2
- net labels removed: MC+, signaling
- wire segments 39 -> 13
- no-connect marks 2 -> 0
Other:
- moved on the sheet: C6
