File: motor controller RS485/motor controller.sch (KiCad schematic (older format))
At the start: 29 parts, among them IC1 MA702, IC2 MC33926PNB, IC3 LP38690SD-ADJ_NOPB, IC4 LTC2850IS8PBF, J1 Conn_01x04_Male, J2 Conn_01x04_Male, J3 Conn_01x04_Male, M1 Motor_DC, U1 STM32L432KCUx, Y1 32mhz

Commit message: Updated RS485 variant
Parts:
- removed C8, C9: 1UF, Capacitor_SMD:C_0402_1005Metric, symbol Device:C
- removed IC3: LP38690SD-ADJ_NOPB, LP38690SD-ADJ_NOPB:SON95P300X300X80-7N, symbol LP38690SD-ADJ_NOPB:LP38690SD-ADJ_NOPB
- removed IC4: LTC2850IS8PBF, LTC2850IS8PBF:SOIC127P600X175-8N, symbol LTC2850IS8PBF:LTC2850IS8PBF
- removed Y1: 32mhz, Crystal:Crystal_SMD_2016-4Pin_2.0x1.6mm, symbol Device:Crystal_GND24
- added IC3: SN65HVD75DRBT, SN65HVD75DRBT:SON65P300X300X100-9N-D, symbol SN65HVD75DRBT:SN65HVD75DRBT
- added U2: MIC5504-3.3YM5, Package_TO_SOT_SMD:SOT-23-5, symbol Regulator_Linear:MIC5504-3.3YM5
- C1, C2: value 10pF -> C
- R3: value 120 -> 10K
Connections:
- wire segments 36 -> 26
Other:
- moved on the sheet: C3, C4, C5, C6, C7, D1, IC1, IC2, J1, J2, J3, M1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
